File: zab-let.sch (KiCad schematic (older format))
At the start: 37 parts, among them J1 CONN_3, J2 CONN_4X2, Q1 BC547, Q2 BC547, Q3 BC547, Q4 BC547, Q5 BC557, SW1 SW_PUSH, U1 ATTINY24-44-84/DIP-SO, X1 RESONATOR

Commit message: Last update from Subversion
Parts:
- C1: value 100µ -> 10u
- R1: value 1K -> 47K
